File: Kolya's Steno Keyboard.kicad_sch (KiCad schematic)
At the start: 0 parts

Commit message: today I learned how to create a schematic, and create a keyboard matrix and how to wire it to a micro controller.
Parts:
- added D1, D2, D3, D4, D5, D6, D7, D8, D9: Diode, symbol ScottoKeebs:Placeholder_Diode
- added S1, S2, S3, S4, S5, S6, S7, S8, S9: Keyswitch, symbol ScottoKeebs:Placeholder_Keyswitch
- added U1: Arduino_Pro_Micro, ScottoKeebs_MCU:Arduino_Pro_Micro, symbol ScottoKeebs:MCU_Arduino_Pro_Micro
Connections:
- new net: D4.2 (A), S4.2
- new net: D5.2 (A), S5.2
- new net: D2.2 (A), S2.2
- new net: D9.2 (A), S9.2
- new net: D6.2 (A), S6.2
- new net: D7.2 (A), S7.2
- new net: D1.2 (A), S1.2
- new net: D3.2 (A), S3.2
- new net: D8.2 (A), S8.2
- new net column0: S1.1, S4.1, S7.1, U1.5 (2/PD1)
- new net column1: S2.1, S5.1, S8.1, U1.6 (3/PD0)
- new net column2: S3.1, S6.1, S9.1, U1.7 (4/PD4)
- new net row0: D1.1 (K), D2.1 (K), D3.1 (K), U1.8 (5/PC6)
- new net row1: D4.1 (K), D5.1 (K), D6.1 (K), U1.9 (6/PD7)
- new net row2: D7.1 (K), D8.1 (K), D9.1 (K), U1.10 (7/PE6)
